File: hardware/bzkhs_sheered_shenzen.kicad_pcb (KiCad board)
At the start: 2 copper layers, 257.5 x 75.4 mm, 3 parts

Commit message: All placed
Parts:
- removed the G*** at (0.00, 0.00) (x3)
- added BT1: Battery_Cell, BZKHS:aaa, B.Cu at (142.1, 45.8)
- added C1: C, Capacitors_SMD:C_0805, B.Cu at (151.7, 37.1)
- added C2: C, Capacitors_SMD:C_0805, B.Cu at (147.9, 45.8)
- added D1: LED, BZKHS:LED, B.Cu at (64.9, 60.8)
- added D10: LED, BZKHS:LED, B.Cu at (240.7, 84.5)
- added D2: LED, BZKHS:LED, B.Cu at (35.6, 82.9)
- added D3: LED, BZKHS:LED, B.Cu at (112.9, 59.1)
- added D4: LED, BZKHS:LED, B.Cu at (82.5, 90.5)
- added D5: LED, BZKHS:LED, B.Cu at (156.7, 60.2)
- added D6: LED, BZKHS:LED, B.Cu at (127.0, 82.6)
- added D7: LED, BZKHS:LED, B.Cu at (214.2, 61.5)
- added D8: LED, BZKHS:LED, B.Cu at (177.9, 81.7)
- added D9: LED, BZKHS:LED, B.Cu at (242.6, 58.2)
- added G*** (x3): LOGO, LOGO, F.Cu at (148.2, 149.7)
- added ICSP1: Conn_01x05, SF_Connectors:1X05_LOCK_LONGPADS, B.Cu at (152.0, 30.4)
- added J1: Conn_01x04, SF_Connectors:1X04_LONGPADS, B.Cu at (180.7, 30.4)
- added J2: Conn_01x04, SF_Connectors:1X04_LONGPADS, B.Cu at (137.5, 30.4)
- added J3: Conn_01x04, SF_Connectors:1X04_LONGPADS, B.Cu at (122.5, 30.2)
- added J4: Conn_01x02, SF_Connectors:1X02_LONGPADS, B.Cu at (109.8, 30.4)
- added J5: Conn_01x02, SF_Connectors:1X02_LONGPADS, B.Cu at (200.9, 30.4)
- added Q1: Q_NPN_BEC, SF_Silicon-Standard:SOT23-3, B.Cu at (219.1, 30.5)
- added Q2: Q_NPN_BEC, SF_Silicon-Standard:SOT23-3, B.Cu at (97.1, 30.4)
- added Q3: Q_NPN_BEC, SF_Silicon-Standard:SOT23-3, B.Cu at (72.4, 54.2)
- added Q4: Q_NPN_BEC, SF_Silicon-Standard:SOT23-3, B.Cu at (112.9, 52.2)
- added Q5: Q_NPN_BEC, SF_Silicon-Standard:SOT23-3, B.Cu at (165.7, 52.3)
- added Q6: Q_NPN_BEC, SF_Silicon-Standard:SOT23-3, B.Cu at (215.3, 51.9)
- added Q7: Q_NPN_BEC, SF_Silicon-Standard:SOT23-3, B.Cu at (236.7, 52.6)
- added R1: 1kR, Resistors_SMD:R_0805, B.Cu at (214.6, 30.5)
- added R10: 50R, Resistors_SMD:R_0805, B.Cu at (118.0, 84.5)
- added R11: 50R, Resistors_SMD:R_0805, B.Cu at (168.8, 82.8)
- added R12: 50R, Resistors_SMD:R_0805, B.Cu at (228.3, 84.1)
- added R2: 1kR, Resistors_SMD:R_0805, B.Cu at (101.5, 30.3)
- added R3: 1kR, Resistors_SMD:R_0805, B.Cu at (73.7, 50.8)
- added R4: 1kR, Resistors_SMD:R_0805, B.Cu at (112.8, 48.5)
- added R5: 1kR, Resistors_SMD:R_0805, B.Cu at (165.7, 48.6)
- added R6: 1kR, Resistors_SMD:R_0805, B.Cu at (215.3, 48.2)
- added R7: 1kR, Resistors_SMD:R_0805, B.Cu at (235.1, 49.1)
- added R8: 50R, Resistors_SMD:R_0805, B.Cu at (43.7, 85.8)
- added R9: 50R, Resistors_SMD:R_0805, B.Cu at (79.5, 78.5)
- added REF**: MountingHole_4mm, Mounting_Holes:MountingHole_4mm, F.Cu at (234.5, 31.6)
- added REF**: MountingHole_4mm, Mounting_Holes:MountingHole_4mm, F.Cu at (81.5, 31.6)
- added SAO1: 2X2, Pin_Headers:Pin_Header_Straight_2x02_Pitch2.54mm, F.Cu at (224.3, 33.1)
- added SAO2: 2X2, Pin_Headers:Pin_Header_Straight_2x02_Pitch2.54mm, F.Cu at (89.2, 33.0)
- added SW1: DPDT, BZKHS:JS202011JAQN, B.Cu at (169.8, 31.9)
- added U1: STM32L031F6, Housings_SSOP:TSSOP-20_4.4x6.5mm_Pitch0.65mm, B.Cu at (156.8, 37.1)
Routing:
- net +3V3: track 0.00 -> 281.0 mm
- net Net-(D7-Pad2): track 0.00 -> 41.7 mm
- net Net-(D3-Pad2): track 0.00 -> 41.4 mm
- net Net-(D5-Pad2): track 0.00 -> 35.9 mm
- net Net-(D1-Pad2): track 0.00 -> 35.4 mm
- net Net-(D10-Pad1): track 0.00 -> 19.6 mm
- net Net-(D10-Pad2): track 0.00 -> 14.1 mm
- net Net-(D5-Pad1): track 0.00 -> 11.2 mm
- net Net-(D6-Pad2): track 0.00 -> 11.1 mm
- net Net-(D8-Pad2): track 0.00 -> 10.5 mm
- net Net-(D1-Pad1): track 0.00 -> 9.22 mm
- net Net-(D2-Pad2): track 0.00 -> 8.48 mm
- net Net-(D7-Pad1): track 0.00 -> 7.45 mm
- net Net-(D9-Pad1): track 0.00 -> 7.15 mm
- net Net-(D4-Pad2): track 0.00 -> 6.81 mm
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- added copper zone on B.Cu, net GND
Other:
- outline, holes or cut-outs redrawn

Commit message: Finished
Parts:
- removed the G*** at (148.2, 149.7) (x2)
- removed J1, J2: Conn_01x04, SF_Connectors:1X04_LONGPADS
- removed J4, J5: Conn_01x02, SF_Connectors:1X02_LONGPADS
- added ?: , BZKHS:bazooka, F.Cu at (226.9, 42.5)
- added ?: , BZKHS:bazooka_text, F.Cu at (172.8, 44.8)
- added ?: , BZKHS:p_logo_5_copper, F.Cu at (78.9, 42.9)
- added F1: Fiducial, SF_Aesthetics:FIDUCIAL-MICRO, F.Cu at (222.5, 28.8)
- added F1: Fiducial, SF_Aesthetics:FIDUCIAL-MICRO, F.Cu at (87.4, 28.6)
- added G*** (x2): LOGO, LOGO, F.Cu at (148.2, 149.7)
- turned R6 to 270 degrees
Routing:
- net /SDA: track 0.00 -> 144.5 mm, vias 0 -> 5
- net /SCL: track 0.00 -> 141.2 mm, vias 0 -> 5
- net /PA6: track 0.00 -> 126.8 mm, vias 0 -> 6
- net /PA1: track 0.00 -> 90.9 mm, vias 0 -> 2
- net /PA5: track 0.00 -> 84.9 mm, vias 0 -> 2
- net GND: track 0.00 -> 82.3 mm, vias 0 -> 6
- net /PA4: track 0.00 -> 58.5 mm, vias 0 -> 2
- net /PA2: track 0.00 -> 50.6 mm
- net /BOOT0: track 0.00 -> 39.1 mm, vias 0 -> 4
- net /PB1: track 0.00 -> 34.0 mm, vias 0 -> 4
- net Net-(BT1-Pad2): track 0.00 -> 23.3 mm
- net /PA3: track 0.00 -> 14.0 mm, vias 0 -> 2
- net +3V3: track 281.0 -> 294.4 mm, vias 0 -> 1
- net Net-(Q2-Pad3): track 0.00 -> 8.55 mm
- net /RST: track 0.00 -> 7.40 mm
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- added copper zone on F.Cu, net +3V3
Other:
- net class HighCurrent added: clearance 0.2, trace_width 0.9, via_dia 0.8, via_drill 0.5
- board text added: "Nyy Nebhaq"
- board text added: "Va Gur Pragre"
